File: PCB/hackpad-v1.kicad_pcb (KiCad board)
At the start: 2 copper layers, 5 parts, among them SW1 SW_Push, SW2 SW_Push, SW3 SW_Push, SW4 RotaryEncoder_Switch, U1 MOUDLE-SEEEDUINO-XIAO

Commit message: fix production files and gerbers for jlc pcb
Routing:
- net Net-(U1-PA9_A5_D5_SCL): track 54.8 -> 62.1 mm
Other:
- board outline added: 22.8 x 75.2 mm
Changed lines of the file:
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@@
 		(filling no)
 		(pcbplotparams
-			(layerselection 0x00000000_00000000_55555555_5755f5ff)
-			(plot_on_all_layers_selection 0x00000000_00000000_00000000_00000000)
+			(layerselection 0x00000000_00000000_55557fdf_ffffffff)
+			(plot_on_all_layers_selection 0x00000000_00000000_00002a8a_aaaaaaaf)
 			(disableapertmacros no)
 			(usegerberextensions no)
@@
 			(dashed_line_gap_ratio 3)
 			(svgprecision 4)
-			(plotframeref no)
+			(plotframeref yes)
 			(mode 1)
 			(useauxorigin no)
@@
 			(outputformat 1)
 			(mirror no)
-			(drillshape 1)
+			(drillshape 0)
 			(scaleselection 1)
-			(outputdirectory "")
+			(outputdirectory "../../hackpad-v1_gerbers-2/")
 		)
 	)
@@
 		(tags "rotary encoder")
 		(property "Reference" "SW4"
-			(at 2.8 -4.7 0)
+			(at 7.7175 -4.895 0)
 			(layer "F.SilkS")
 			(effects
@@
 		)
 		(fp_text user "${REFERENCE}"
-			(at 11.1 6.3 0)
+			(at 7.5 6.25 0)
 			(layer "F.Fab")
 			(effects
@@
 		(embedded_fonts no)
 	)
+	(gr_rect
+		(start 110.435 120.105)
+		(end 129.5 136.25)
+		(stroke
+			(width 0.1)
+			(type default)
+		)
+		(fill no)
+		(layer "Dwgs.User")
+	)
+	(gr_rect
+		(start 108.5 61.5)
+		(end 131.25 136.75)
+		(stroke
+			(width 0.05)
+			(type default)
+		)
+		(fill no)
+		(layer "Edge.Cuts")
+	)
 	(gr_text "Bye bye Nathan,\n we'll never forget you:)\nand yeah, you are\n NotARoomba"
 		(at 120.5 99 0)
@@
 	)
 	(segment
-		(start 122.5 105.5)
-		(end 122.5 88.623654)
+		(start 122.5 88.91)
+		(end 112.25 78.66)
 		(width 0.2)
 		(layer "B.Cu")
@@
 	)
 	(segment
-		(start 122.5 88.623654)
-		(end 112.536346 78.66)
+		(start 112.536346 78.66)
+		(end 112.25 78.66)
 		(width 0.2)
 		(layer "B.Cu")
@@
 	)
 	(segment
-		(start 112.536346 78.66)
-		(end 112.25 78.66)
+		(start 122.5 105.5)
+		(end 122.5 88.91)
 		(width 0.2)
 		(layer "B.Cu")
@@
 	)
 	(segment
-		(start 116.11 69.96)
-		(end 116.11 92.89)
+		(start 112.25 68.5)
+		(end 113.71 69.96)
 		(width 0.2)
 		(layer "F.Cu")
@@
 	)
 	(segment
-		(start 126.75 125)
-		(end 116.15 114.4)
+		(start 113.71 69.96)
+		(end 116.11 69.96)
 		(width 0.2)
 		(layer "F.Cu")
@@
 	)
 	(segment
-		(start 116.11 92.89)
-		(end 116.15 92.93)
+		(start 116.11 69.96)
+		(end 116.11 76.39)
 		(width 0.2)
 		(layer "F.Cu")
@@
 	)
 	(segment
-		(start 116.15 92.93)
-		(end 116.15 108.04)
+		(start 116.11 76.39)
+		(end 116.15 76.43)
 		(width 0.2)
 		(layer "F.Cu")
@@
 	)
 	(segment
-		(start 116.11 69.96)
-		(end 114.65 68.5)
+		(start 126.75 125)
+		(end 116.15 114.4)
 		(width 0.2)
-		(layer "B.Cu")
+		(layer "F.Cu")
 		(net "GND")
 	)
 	(segment
-		(start 114.65 68.5)
-		(end 112.25 68.5)
+		(start 116.15 76.43)
+		(end 116.15 108.04)
 		(width 0.2)
-		(layer "B.Cu")
+		(layer "F.Cu")
 		(net "GND")
 	)
@@
 	)
 	(segment
+		(start 127.5 71.04)
+		(end 127.5 71)
+		(width 0.2)
+		(layer "F.Cu")
+		(net "Net-(U1-PA10_A2_D2)")
+	)
+	(segment
 		(start 123.928629 90.428629)
 		(end 123.44 90.917258)
@@
 	)
 	(segment
-		(start 127.5 71.04)
-		(end 127.5 72)
-		(width 0.2)
-		(layer "B.Cu")
-		(net "Net-(U1-PA10_A2_D2)")
-	)
-	(segment
 		(start 124 105.020101)
 		(end 124 106.5)
@@
 	)
 	(segment
-		(start 127.5 72)
-		(end 123.928629 75.571371)
+		(start 124 106.5)
+		(end 122.27 108.23)
 		(width 0.2)
 		(layer "B.Cu")
@@
 	)
 	(segment
-		(start 124 106.5)
-		(end 122.27 108.23)
+		(start 127.5 71.04)
+		(end 127.5 72)
 		(width 0.2)
 		(layer "B.Cu")
@@
 	)
 	(segment
-		(start 124.542944 92.78)
-		(end 123.84 92.077056)
+		(start 127.5 72)
+		(end 123.928629 75.571371)
 		(width 0.2)
 		(layer "B.Cu")
-		(net "Net-(U1-PA11_A3_D3)")
+		(net "Net-(U1-PA10_A2_D2)")
 	)
 	(segment
-		(start 126 75.08)
-		(end 127.5 73.58)
+		(start 124.542944 92.78)
+		(end 123.84 92.077056)
 		(width 0.2)
 		(layer "B.Cu")
@@
 	)
 	(segment
+		(start 127.5 73.58)
+		(end 126 75.08)
+		(width 0.2)
+		(layer "B.Cu")
+		(net "Net-(U1-PA11_A3_D3)")
+	)
+	(segment
 		(start 123.84 91.082944)
 		(end 126 88.922944)
@@
 	)
 	(segment
-		(start 130.6 126.15)
-		(end 126.75 130)
+		(start 117.61 103.36)
+		(end 117.61 88.55)
 		(width 0.2)
-		(layer "B.Cu")
+		(layer "F.Cu")
 		(net "Net-(U1-PA9_A5_D5_SCL)")
 	)
 	(segment
-		(start 127.5 78.66)
-		(end 128.536346 78.66)
+		(start 129 119.75)
+		(end 123.25 114)
 		(width 0.2)
-		(layer "B.Cu")
+		(layer "F.Cu")
 		(net "Net-(U1-PA9_A5_D5_SCL)")
 	)
 	(segment
-		(start 128.536346 78.66)
-		(end 130.6 80.723654)
+		(start 117.61 88.55)
+		(end 127.5 78.66)
 		(width 0.2)
-		(layer "B.Cu")
+		(layer "F.Cu")
 		(net "Net-(U1-PA9_A5_D5_SCL)")
 	)
 	(segment
-		(start 130.6 80.723654)
-		(end 130.6 126.15)
+		(start 123.25 114)
+		(end 123.25 109)
+		(width 0.2)
+		(layer "F.Cu")
+		(net "Net-(U1-PA9_A5_D5_SCL)")
+	)
+	(segment
+		(start 129 127.75)
+		(end 129 119.75)
+		(width 0.2)
+		(layer "F.Cu")
+		(net "Net-(U1-PA9_A5_D5_SCL)")
+	)
+	(segment
+		(start 123.25 109)
+		(end 117.61 103.36)
+		(width 0.2)
+		(layer "F.Cu")
+		(net "Net-(U1-PA9_A5_D5_SCL)")
+	)
+	(segment
+		(start 126.75 130)
+		(end 129 127.75)
+		(width 0.2)
+		(layer "F.Cu")
+		(net "Net-(U1-PA9_A5_D5_SCL)")
+	)
+	(segment
+		(start 127.5 78.66)
+		(end 128.536346 78.66)
 		(width 0.2)
 		(layer "B.Cu")
